File: creativision-clone.kicad_sch (KiCad schematic)
At the start: 74 parts, among them J1 Conn_01x10_Socket, J2 Conn_01x10_Socket, J3 Conn_01x03_Socket, P1 Cartridge Slot, SW1 Reset, U1 AS6C62256-DIP, U100 74HCT574, U101 74HCT574, U102 74HCT574, U12 74LS32, U15 74LS139, U18 AS6C62256-DIP, U2 6502, U20 27256, U21 6821, U22 SN76489AN, U3 TMS9918A, U99 74HCT04, X1 2MHz

Commit message: Wire 30
Parts:
- added C3: 10µF, symbol Device:C_Polarized_Small_US
- added R27, R68: 3.3kΩ, symbol Device:R_Small_US
Connections:
- net AUDIO_IN: now reaches P1.30 (Pin_30)
- net AUDIO_IN: now also C3.1
- net COMVID: now reaches U3.36 (COMVID)
- net PSG_OUT: now reaches U22.7 (Audio)
- net PSG_OUT: now also R68.1
- new net: R27.2, R68.2
- new net: C3.2, R27.1
Other:
- note added: "A/V Out"
- note removed: "TODO: What does pin 30 do?"
Changed lines of the file:
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@@
   (junction (at 310.515 73.025) (diameter 0) (color 0 0 0 0)
   )
+  (junction (at 325.755 165.735) (diameter 0) (color 0 0 0 0)
+  )
   (junction (at 329.565 74.295) (diameter 0) (color 0 0 0 0)
   )
@@
     (stroke (width 0) (type default))
   )
+  (wire (pts (xy 289.56 113.665) (xy 289.56 165.735))
+    (stroke (width 0) (type default))
+  )
   (wire (pts (xy 215.9 85.09) (xy 215.9 93.345))
     (stroke (width 0) (type default))
@@
     (stroke (width 0) (type default))
   )
+  (wire (pts (xy 289.56 165.735) (xy 315.595 165.735))
+    (stroke (width 0) (type default))
+  )
   (wire (pts (xy 226.695 139.065) (xy 226.695 143.51))
     (stroke (width 0) (type default))
@@
     (stroke (width 0) (type default))
   )
+  (wire (pts (xy 232.41 210.185) (xy 253.365 210.185))
+    (stroke (width 0) (type default))
+  )
   (wire (pts (xy 356.87 73.025) (xy 356.87 53.34))
     (stroke (width 0) (type default))
@@
     (stroke (width 0) (type default))
   )
+  (wire (pts (xy 320.675 165.735) (xy 325.755 165.735))
+    (stroke (width 0) (type default))
+  )
+  (wire (pts (xy 311.785 156.21) (xy 314.96 156.21))
+    (stroke (width 0) (type default))
+  )
   (wire (pts (xy 307.975 85.725) (xy 307.975 80.645))
     (stroke (width 0) (type default))
@@
     (stroke (width 0) (type default))
   )
+  (wire (pts (xy 320.04 156.21) (xy 325.755 156.21))
+    (stroke (width 0) (type default))
+  )
   (wire (pts (xy 353.695 29.21) (xy 353.695 26.035))
     (stroke (width 0) (type default))
@@
     (stroke (width 0) (type default))
   )
+  (wire (pts (xy 86.995 238.125) (xy 102.235 238.125))
+    (stroke (width 0) (type default))
+  )
   (wire (pts (xy 348.615 29.21) (xy 342.9 29.21))
     (stroke (width 0) (type default))
@@
     (stroke (width 0) (type default))
   )
+  (wire (pts (xy 79.375 244.475) (xy 86.995 244.475))
+    (stroke (width 0) (type default))
+  )
   (wire (pts (xy 271.78 45.72) (xy 271.78 45.085))
     (stroke (width 0) (type default))
@@
     (stroke (width 0) (type default))
   )
+  (wire (pts (xy 302.26 156.21) (xy 306.705 156.21))
+    (stroke (width 0) (type default))
+  )
   (wire (pts (xy 256.54 106.045) (xy 256.54 109.855))
     (stroke (width 0) (type default))
@@
     (stroke (width 0) (type default))
   )
+  (wire (pts (xy 319.405 113.665) (xy 289.56 113.665))
+    (stroke (width 0) (type default))
+  )
   (wire (pts (xy 32.385 170.18) (xy 35.56 170.18))
     (stroke (width 0) (type default))
@@
     (stroke (width 0) (type default))
   )
+  (wire (pts (xy 325.755 156.21) (xy 325.755 165.735))
+    (stroke (width 0) (type default))
+  )
   (wire (pts (xy 129.54 57.15) (xy 141.605 57.15))
     (stroke (width 0) (type default))
@@
     (stroke (width 0) (type default))
   )
+  (wire (pts (xy 325.755 165.735) (xy 342.9 165.735))
+    (stroke (width 0) (type default))
+  )
   (wire (pts (xy 292.1 54.61) (xy 287.655 54.61))
     (stroke (width 0) (type default))
@@
     (stroke (width 0) (type default))
   )
+  (wire (pts (xy 86.995 244.475) (xy 86.995 238.125))
+    (stroke (width 0) (type default))
+  )
   (wire (pts (xy 269.24 65.405) (xy 297.18 65.405))
     (stroke (width 0) (type default))
@@
     (stroke (width 0) (type default))
   )
-  (text "TODO: Wire up audio out" (at 346.075 126.365 0)
+  (rectangle (start 283.21 146.05) (end 365.125 197.485)
+    (stroke (width 0) (type dot))
+    (fill (type none))
+  )
+  (text "TODO: Wire up audio out" (at 354.33 158.115 0)
     (effects (font (size 1.27 1.27)) (justify right bottom))
   )
@@
     (effects (font (size 1.27 1.27)) (justify left bottom))
   )
-  (text "TODO: What does pin 30 do?" (at 250.19 201.93 0)
-    (effects (font (size 1.27 1.27)) (justify left bottom))
-  )
   (text "TODO: Which project is it that I had the dual footprint oscillator in?"
     (at 36.195 19.685 0)
@@
     (effects (font (size 1.27 1.27) bold) (justify right bottom))
   )
-  (text "TODO: Video out amplification" (at 88.9 224.79 0)
+  (text "TODO: Video out amplification" (at 357.505 186.69 0)
     (effects (font (size 1.27 1.27)) (justify right bottom))
   )
+  (text "A/V Out" (at 354.33 149.86 0)
+    (effects (font (size 1.27 1.27) (thickness 0.254) bold) (justify left bottom))
+  )
   (label "~{ROM_RD}" (at 242.57 215.265 0) (fields_autoplaced)
     (effects (font (size 1.27 1.27)) (justify left bottom))
@@
     (effects (font (size 1.27 1.27)) (justify left bottom))
   )
+  (label "PSG_OUT" (at 302.26 165.735 180) (fields_autoplaced)
+    (effects (font (size 1.27 1.27)) (justify right bottom))
+  )
   (label "d0" (at 243.84 40.005 180) (fields_autoplaced)
     (effects (font (size 1.27 1.27)) (justify right bottom))
@@
     (effects (font (size 1.27 1.27)) (justify right bottom))
   )
+  (label "COMVID" (at 102.235 238.125 0) (fields_autoplaced)
+    (effects (font (size 1.27 1.27)) (justify left bottom))
+  )
   (label "PA2" (at 332.74 45.72 180) (fields_autoplaced)
     (effects (font (size 1.27 1.27)) (justify right bottom))
@@
     (effects (font (size 1.27 1.27)) (justify right bottom))
   )
+  (label "AUDIO_IN" (at 302.26 156.21 180) (fields_autoplaced)
+    (effects (font (size 1.27 1.27)) (justify right bottom))
+  )
   (label "~{WRAM_OE}" (at 186.69 101.6 0) (fields_autoplaced)
     (effects (font (size 1.27 1.27)) (justify left bottom))
@@
     (effects (font (size 1.27 1.27)) (justify right bottom))
   )
+  (label "AUDIO_IN" (at 253.365 210.185 0) (fields_autoplaced)
+    (effects (font (size 1.27 1.27)) (justify left bottom))
+  )
   (label "d2" (at 62.23 130.81 0) (fields_autoplaced)
     (effects (font (size 1.27 1.27)) (justify left bottom))
@@
     (effects (font (size 1.27 1.27)) (justify right bottom))
   )
+  (label "COMVID" (at 291.465 179.705 180) (fields_autoplaced)
+    (effects (font (size 1.27 1.27)) (justify right bottom))
+  )
   (label "vd3" (at 79.375 262.255 0) (fields_autoplaced)
     (effects (font (size 1.27 1.27)) (justify left bottom))
@@
     )
   )
+  (symbol (lib_id "Device:R_Small_US") (at 318.135 165.735 90) (unit 1)
+    (in_bom yes) (on_board yes) (dnp no) (fields_autoplaced)
+    (property "Reference" "R68" (at 318.135 161.29 90)
+      (effects (font (size 1.27 1.27)))
+    )
+    (property "Value" "3.3kΩ" (at 318.135 163.83 90)
+      (effects (font (size 1.27 1.27)))
+    )
+    (property "Footprint" "" (at 318.135 165.735 0)
+      (effects (font (size 1.27 1.27)) hide)
+    )
+    (property "Datasheet" "~" (at 318.135 165.735 0)
+      (effects (font (size 1.27 1.27)) hide)
+    )
+    (pin "1")
+    (pin "2")
+    (instances
+      (project "creativision-clone"
+        (path "/4f154aad-bddd-4366-bec7-a527fffe24b1"
+          (reference "R68") (unit 1)
+        )
+      )
+    )
+  )
   (symbol (lib_id "Device:D_Small") (at 326.39 27.94 180) (unit 1)
     (in_bom yes) (on_board yes) (dnp no)
@@
     )
   )
+  (symbol (lib_id "Device:R_Small_US") (at 317.5 156.21 90) (unit 1)
+    (in_bom yes) (on_board yes) (dnp no) (fields_autoplaced)
+    (property "Reference" "R27" (at 317.5 151.13 90)
+      (effects (font (size 1.27 1.27)))
+    )
+    (property "Value" "3.3kΩ" (at 317.5 153.67 90)
+      (effects (font (size 1.27 1.27)))
+    )
+    (property "Footprint" "" (at 317.5 156.21 0)
+      (effects (font (size 1.27 1.27)) hide)
+    )
+    (property "Datasheet" "~" (at 317.5 156.21 0)
+      (effects (font (size 1.27 1.27)) hide)
+    )
+    (pin "1")
+    (pin "2")
+    (instances
+      (project "creativision-clone"
+        (path "/4f154aad-bddd-4366-bec7-a527fffe24b1"
+          (reference "R27") (unit 1)
+        )
+      )
+    )
+  )
   (symbol (lib_id "74xx:74HCT04") (at 84.455 336.55 0) (unit 3)
     (in_bom yes) (on_board yes) (dnp no) (fields_autoplaced)
@@
         )
       )
+    )
+  )
+  (symbol (lib_id "Device:C_Polarized_Small_US") (at 309.245 156.21 90) (unit 1)
+    (in_bom yes) (on_board yes) (dnp no) (fields_autoplaced)
+    (property "Reference" "C3" (at 308.8132 151.13 90)
+      (effects (font (size 1.27 1.27)))
+    )
+    (property "Value" "10µF" (at 308.8132 153.67 90)
+      (effects (font (size 1.27 1.27)))
+    )
+    (property "Footprint" "" (at 309.245 156.21 0)
+      (effects (font (size 1.27 1.27)) hide)
+    )
+    (property "Datasheet" "~" (at 309.245 156.21 0)
+      (effects (font (size 1.27 1.27)) hide)
+    )
+    (pin "1")
+    (pin "2")
+    (instances
+      (project "creativision-clone"
+        (path "/4f154aad-bddd-4366-bec7-a527fffe24b1"
+          (reference "C3") (unit 1)
+        )
+      )

Commit message: J3: Cassette interface
Parts:
- removed J3: Conn_01x03_Socket, symbol Connector:Conn_01x03_Socket
- added D17: LED, symbol Device:LED
- added J3: Conn_01x07_Pin, symbol Connector:Conn_01x07_Pin
- added J4: Conn_01x04_Socket, symbol Connector:Conn_01x04_Socket
- added JP6: SolderJumper_3_Bridged12, symbol Jumper:SolderJumper_3_Bridged12
- added R2: 330Ω, symbol Device:R_Small_US
Connections:
- net +12V: now also J4.2 (Pin_2)
- net +5V: now also D17.2 (A), JP6.3 (B)
- net -5V: now also J4.1 (Pin_1)
- net AUDIO_IN: now also J3.1 (Pin_1)
- net GND: now also J3.7 (Pin_7), J4.4 (Pin_4), R2.2
- net PA4: now reaches U21.6 (PA4)
- net PA4: now also J3.5 (Pin_5)
- net PA5: now reaches U21.7 (PA5)
- net PA5: now also J3.4 (Pin_4)
- net PA6: now reaches U21.8 (PA6)
- net PA6: now also J3.3 (Pin_3)
- net PA7: now reaches U21.9 (PA7)
- net PA7: now also J3.2 (Pin_2)
- new net: D17.1 (K), R2.1
- new net +9V: J4.3 (Pin_3), JP6.1 (A)
- new net TAPE_VCC: J3.6 (Pin_6), JP6.2 (C)
Other:
- note added: "Optional power injection (for carts that need -5V, 12V, tape that needs 9V)"
- note added: "TODO: Connector J3?"
- note added: "Tape interface"
- note removed: "Optional power injection (for carts that need -5V, 12V)"
- note removed: "TODO: Connector P1?"
- note removed: "TODO: J3"
