File: creativision-clone.kicad_sch (KiCad schematic)
At the start: 108 parts, among them J1 Conn_01x10_Socket, J2 Conn_01x10_Socket, J3 Conn_01x07_Pin, J4 Conn_01x04_Socket, J5 RCJ-013, J6 RCJ-014, P1 Cartridge Slot, Q1 2n4401, SW1 Reset, SW2 Power Toggle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

Commit message: Footprints except cart
Parts:
- P1: DigiKey (none) -> 2-5530843-7-ND
Changed lines of the file:
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@@
+      (effects (font (size 1.27 1.27)) hide)
+    )
+    (property "DigiKey" "2-5530843-7-ND" (at 224.79 194.945 0)
       (effects (font (size 1.27 1.27)) hide)
     )

Commit message: Partial layout
Parts:
- U3: footprint Package_DIP:DIP-40_W25.4mm_Socket_LongPads -> Package_DIP:DIP-40_W15.24mm_Socket_LongPads
Changed lines of the file:
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@@
       (effects (font (size 1.27 1.27)))
     )
-    (property "Footprint" "Package_DIP:DIP-40_W25.4mm_Socket_LongPads" (at 66.675 229.235 0)
+    (property "Footprint" "Package_DIP:DIP-40_W15.24mm_Socket_LongPads" (at 66.675 229.235 0)
       (effects (font (size 1.27 1.27)) hide)
     )

Commit message: Enough for one night
Parts:
- removed C10, C106, C11: 100µF, Capacitor_THT:CP_Radial_D6.3mm_P2.50mm, symbol Device:C_Polarized_Small_US
- removed JP1, JP2, JP3, JP4: SolderJumper_2_Bridged, Jumper:SolderJumper-2_P1.3mm_Bridged2Bar_RoundedPad1.0x1.5mm, symbol Jumper:SolderJumper_2_Bridged
Connections:
- net GND: now also U20.2 (A12), U20.23 (A11), U20.26 (A13), U20.27 (A14)
- net SW_VCC: now reaches C13.2, SW2.2
Other:
- note added: "TODO: Which value to use?"

Commit message: Fix backwards tape header
Connections:
- net AUDIO_IN: now also J3.7 (Pin_7); no longer J3.1 (Pin_1)
- net GND: now also J3.1 (Pin_1); no longer J3.7 (Pin_7)
- net PA4: now also J3.3 (Pin_3); no longer J3.5 (Pin_5)
- net PA6: now also J3.5 (Pin_5); no longer J3.3 (Pin_3)
- net PA7: now also J3.6 (Pin_6); no longer J3.2 (Pin_2)
- net TAPE_VCC: now also J3.2 (Pin_2); no longer J3.6 (Pin_6)
Other:
- moved on the sheet: J3
Changed lines of the file:
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@@
     )
   )
-  (symbol (lib_id "Connector:Conn_01x07_Pin") (at 297.815 219.075 0) (mirror y) (unit 1)
-    (in_bom yes) (on_board yes) (dnp no) (fields_autoplaced)
-    (property "Reference" "J3" (at 299.72 218.44 0)
+  (symbol (lib_id "Connector:Conn_01x07_Pin") (at 297.815 219.075 180) (unit 1)
+    (in_bom yes) (on_board yes) (dnp no)
+    (property "Reference" "J3" (at 299.72 219.71 0)
       (effects (font (size 1.27 1.27)) (justify right))
     )
-    (property "Value" "Conn_01x07_Pin" (at 299.72 220.98 0)
+    (property "Value" "Conn_01x07_Pin" (at 299.72 217.17 0)
       (effects (font (size 1.27 1.27)) (justify right))
     )

Commit message: Ugly cartridge connector
Parts:
- P1: footprint (none) -> CreatiVision:Cartridge_Slot_36p
Changed lines of the file:
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@@
       (effects (font (size 1.27 1.27)))
     )
-    (property "Footprint" "" (at 224.79 194.945 0)
+    (property "Footprint" "CreatiVision:Cartridge_Slot_36p" (at 224.79 194.945 0)
       (effects (font (size 1.27 1.27)) hide)
     )

Commit message: Add jumper to default 27c64 pin 27 to high
Parts:
- added JP1: 27c64_Select, Jumper:SolderJumper-3_P1.3mm_Bridged12_RoundedPad1.0x1.5mm_NumberLabels, symbol Jumper:SolderJumper_3_Bridged12
Connections:
- net +5V: now also JP1.1 (A)
- net GND: now also JP1.3 (B); no longer U20.27 (A14)
- new net BIOS_A14: JP1.2 (C), U20.27 (A14)
Changed lines of the file:
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@@
   (junction (at 310.515 27.94) (diameter 0) (color 0 0 0 0)
   )
+  (junction (at 13.335 153.67) (diameter 0) (color 0 0 0 0)
+  )
   (junction (at 353.695 38.735) (diameter 0) (color 0 0 0 0)
   )
@@
   (junction (at 371.475 79.375) (diameter 0) (color 0 0 0 0)
   )
-  (junction (at 13.335 161.29) (diameter 0) (color 0 0 0 0)
-  )
   (junction (at 96.52 140.335) (diameter 0) (color 0 0 0 0)
   )
@@
   )
   (junction (at 342.9 165.735) (diameter 0) (color 0 0 0 0)
+  )
+  (junction (at 52.07 120.65) (diameter 0) (color 0 0 0 0)
   )
   (junction (at 353.695 41.91) (diameter 0) (color 0 0 0 0)
@@
     (stroke (width 0) (type default))
   )
+  (wire (pts (xy 19.05 145.415) (xy 13.335 145.415))
+    (stroke (width 0) (type default))
+  )
   (wire (pts (xy 328.93 61.595) (xy 329.565 61.595))
     (stroke (width 0) (type default))
@@
     (stroke (width 0) (type default))
   )
+  (wire (pts (xy 24.13 149.225) (xy 24.13 161.29))
+    (stroke (width 0) (type default))
+  )
   (wire (pts (xy 95.25 138.43) (xy 95.25 140.335))
     (stroke (width 0) (type default))
@@
     (stroke (width 0) (type default))
   )
+  (wire (pts (xy 24.13 161.29) (xy 41.91 161.29))
+    (stroke (width 0) (type default))
+  )
   (wire (pts (xy 65.405 215.9) (xy 53.975 215.9))
     (stroke (width 0) (type default))
@@
     (stroke (width 0) (type default))
   )
-  (wire (pts (xy 13.335 161.29) (xy 41.91 161.29))
-    (stroke (width 0) (type default))
-  )
   (wire (pts (xy 232.41 194.945) (xy 242.57 194.945))
     (stroke (width 0) (type default))
@@
     (stroke (width 0) (type default))
   )
+  (wire (pts (xy 34.925 145.415) (xy 34.925 120.65))
+    (stroke (width 0) (type default))
+  )
   (wire (pts (xy 353.695 46.355) (xy 371.475 46.355))
     (stroke (width 0) (type default))
@@
     (stroke (width 0) (type default))
   )
-  (wire (pts (xy 13.335 161.29) (xy 13.335 166.37))
-    (stroke (width 0) (type default))
-  )
   (wire (pts (xy 353.695 35.56) (xy 353.695 32.385))
     (stroke (width 0) (type default))
@@
     (stroke (width 0) (type default))
   )
+  (wire (pts (xy 29.21 145.415) (xy 34.925 145.415))
+    (stroke (width 0) (type default))
+  )
   (wire (pts (xy 310.515 59.055) (xy 310.515 73.025))
     (stroke (width 0) (type default))
@@
     (stroke (width 0) (type default))
   )
+  (wire (pts (xy 13.335 145.415) (xy 13.335 153.67))
+    (stroke (width 0) (type default))
+  )
   (wire (pts (xy 79.375 165.735) (xy 79.375 168.91))
     (stroke (width 0) (type default))
@@
     (stroke (width 0) (type default))
   )
-  (wire (pts (xy 13.335 158.75) (xy 13.335 161.29))
+  (wire (pts (xy 13.335 158.75) (xy 13.335 166.37))
     (stroke (width 0) (type default))
   )
@@
   )
   (wire (pts (xy 367.665 165.735) (xy 375.92 165.735))
+    (stroke (width 0) (type default))
+  )
+  (wire (pts (xy 34.925 120.65) (xy 52.07 120.65))
     (stroke (width 0) (type default))
   )
@@
   (label "PA4" (at 292.735 221.615 180) (fields_autoplaced)
     (effects (font (size 1.27 1.27)) (justify right bottom))
+  )
+  (label "BIOS_A14" (at 24.765 161.29 0) (fields_autoplaced)
+    (effects (font (size 1.27 1.27)) (justify left bottom))
   )
   (label "a7" (at 113.03 86.36 0) (fields_autoplaced)
@@
         )
       )
+    )
+  )
+  (symbol (lib_id "Jumper:SolderJumper_3_Bridged12") (at 24.13 145.415 0) (mirror y) (unit 1)
+    (in_bom yes) (on_board yes) (dnp no)
+    (property "Reference" "JP1" (at 24.13 140.97 0)
+      (effects (font (size 1.27 1.27)))
+    )
+    (property "Value" "27c64_Select" (at 24.13 143.51 0)
+      (effects (font (size 1.27 1.27)))
+    )
+    (property "Footprint" "Jumper:SolderJumper-3_P1.3mm_Bridged12_RoundedPad1.0x1.5mm_NumberLabels" (at 24.13 145.415 0)
+      (effects (font (size 1.27 1.27)) hide)
+    )
+    (property "Datasheet" "~" (at 24.13 145.415 0)
+      (effects (font (size 1.27 1.27)) hide)
+    )
+    (pin "1")
+    (pin "2")
+    (pin "3")
+    (instances
+      (project "creativision-clone"
+        (path "/4f154aad-bddd-4366-bec7-a527fffe24b1"
+          (reference "JP1") (unit 1)
+        )
+      )

Commit message: Flip polarity of series filter cap
Connections:
- net +5V: now also C13.2; no longer C13.1
- net SW_VCC: now also C13.1; no longer C13.2
Other:
- note removed: "TODO: are there alternative roms we might want to run?"
- moved on the sheet: C13
Changed lines of the file:
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@@
     (effects (font (size 1.27 1.27)) (justify right bottom))
-  )
-  (text "TODO: are there alternative roms we might want to run?"
-    (at 14.605 186.69 0)
-    (effects (font (size 1.27 1.27)) (justify left bottom))
   )
   (text "VDP" (at 42.545 232.41 0)
@@
     )
   )
-  (symbol (lib_id "Device:C_Polarized_Small_US") (at 153.035 213.995 270) (unit 1)
-    (in_bom yes) (on_board yes) (dnp no) (fields_autoplaced)
-    (property "Reference" "C13" (at 153.4668 208.28 90)
-      (effects (font (size 1.27 1.27)))
-    )
-    (property "Value" "220µF" (at 153.4668 210.82 90)
-      (effects (font (size 1.27 1.27)))
-    )
+  (symbol (lib_id "Device:C_Polarized_Small_US") (at 153.035 213.995 90) (mirror x) (unit 1)
+    (in_bom yes) (on_board yes) (dnp no)
+    (property "Reference" "C13" (at 152.6032 208.28 90)
+      (effects (font (size 1.27 1.27)))
+    )
+    (property "Value" "220µF" (at 152.6032 210.82 90)
+      (effects (font (size 1.27 1.27)))
+    )

Commit message: Delete series filter cap (thanks ZephyrZ80)
Parts:
- removed C13: 220µF, Capacitor_THT:CP_Radial_D6.3mm_P2.50mm, symbol Device:C_Polarized_Small_US
- J5, J6: footprint Jacks:CUI_RCJ-017 -> CUI_RCJ-017
- U1, U18: footprint Package_DIP:DIP-28_W15.24mm_Socket_LongPads -> Housings_DIP:DIP-28_W15.24mm_Socket_LongPads
- U3: footprint Package_DIP:DIP-40_W15.24mm_Socket_LongPads -> Housings_DIP:DIP-40_W15.24mm_Socket_LongPads
- X2: footprint USB-B1HSB6:OST_USB-B1HSB6 -> OST_USB-B1HSB6
Connections:
- net SW_VCC is gone; now on net +5V: SW2.2
Changed lines of the file:
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@@
     (stroke (width 0) (type default))
   )
-  (wire (pts (xy 155.575 213.995) (xy 158.115 213.995))
-    (stroke (width 0) (type default))
-  )
   (wire (pts (xy 331.47 69.215) (xy 332.74 69.215))
     (stroke (width 0) (type default))
@@
     (stroke (width 0) (type default))
   )
-  (wire (pts (xy 140.335 213.995) (xy 150.495 213.995))
+  (wire (pts (xy 140.335 213.995) (xy 158.115 213.995))
     (stroke (width 0) (type default))
   )
@@
       (effects (font (size 1.27 1.27)))
     )
-    (property "Footprint" "Package_DIP:DIP-28_W15.24mm_Socket_LongPads" (at 157.48 104.14 0)
+    (property "Footprint" "Housings_DIP:DIP-28_W15.24mm_Socket_LongPads" (at 157.48 104.14 0)
       (effects (font (size 1.27 1.27)) hide)
     )
@@
       (effects (font (size 1.27 1.27)) (justify right))
     )
-    (property "Footprint" "Jacks:CUI_RCJ-017" (at 383.54 187.325 0)
+    (property "Footprint" "CUI_RCJ-017" (at 383.54 187.325 0)
       (effects (font (size 1.27 1.27)) (justify left bottom) hide)
     )
@@
     )
   )
-  (symbol (lib_id "Device:C_Polarized_Small_US") (at 153.035 213.995 90) (mirror x) (unit 1)
-    (in_bom yes) (on_board yes) (dnp no)
-    (property "Reference" "C13" (at 152.6032 208.28 90)
-      (effects (font (size 1.27 1.27)))
-    )
-    (property "Value" "220µF" (at 152.6032 210.82 90)
-      (effects (font (size 1.27 1.27)))
-    )
-    (property "Footprint" "Capacitor_THT:CP_Radial_D6.3mm_P2.50mm" (at 153.035 213.995 0)
-      (effects (font (size 1.27 1.27)) hide)
-    )
-    (property "Datasheet" "~" (at 153.035 213.995 0)
-      (effects (font (size 1.27 1.27)) hide)
-    )
-    (pin "1")
-    (pin "2")
-    (instances
-      (project "creativision-clone"
-        (path "/4f154aad-bddd-4366-bec7-a527fffe24b1"
-          (reference "C13") (unit 1)
-        )
-      )
-    )
-  )
   (symbol (lib_id "power:GND") (at 52.07 176.53 0) (unit 1)
     (in_bom yes) (on_board yes) (dnp no) (fields_autoplaced)
@@
       (effects (font (size 1.27 1.27)))
     )
-    (property "Footprint" "USB-B1HSB6:OST_USB-B1HSB6" (at 104.775 209.55 0)
+    (property "Footprint" "OST_USB-B1HSB6" (at 104.775 209.55 0)
       (effects (font (size 1.27 1.27)) (justify left bottom) hide)
     )
@@
       (effects (font (size 1.27 1.27)))
     )
-    (property "Footprint" "Package_DIP:DIP-28_W15.24mm_Socket_LongPads" (at 248.285 261.62 0)
+    (property "Footprint" "Housings_DIP:DIP-28_W15.24mm_Socket_LongPads" (at 248.285 261.62 0)
       (effects (font (size 1.27 1.27)) hide)
     )
@@
       (effects (font (size 1.27 1.27)))
     )
-    (property "Footprint" "Jacks:CUI_RCJ-017" (at 383.54 168.275 0)
+    (property "Footprint" "CUI_RCJ-017" (at 383.54 168.275 0)
       (effects (font (size 1.27 1.27)) (justify left bottom) hide)
     )
@@
       (effects (font (size 1.27 1.27)))
     )
-    (property "Footprint" "Package_DIP:DIP-40_W15.24mm_Socket_LongPads" (at 66.675 229.235 0)
+    (property "Footprint" "Housings_DIP:DIP-40_W15.24mm_Socket_LongPads" (at 66.675 229.235 0)
       (effects (font (size 1.27 1.27)) hide)
     )
