File: creativision-clone.kicad_pcb (KiCad board)
At the start: 2 copper layers, 205.7 x 99.7 mm, 102 parts, among them J1 Conn_01x10_Socket, J2 Conn_01x10_Socket, J3 Conn_01x07_Pin, J4 Conn_01x04_Socket, J5 RCJ-013, J6 RCJ-014, Q1 2n4401, SW1 Reset, SW2 Power Toggle, U1 AS6C62256-DIP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

Commit message: Ugly cartridge connector
Parts:
- added P1: Cartridge Slot, CreatiVision:Cartridge_Slot_36p, F.Cu at (73.4, 71.8)
Routing:
- net Net-(X2-VCC): track 81.3 -> 7.50 mm
Changed lines of the file:
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@@
     )
+  )
+  (footprint "CreatiVision:Cartridge_Slot_36p" (layer "F.Cu")
+    (at 73.407 71.781929 -90)
+    (property "DigiKey" "2-5530843-7-ND")
+    (property "Sheetfile" "creativision-clone.kicad_sch")
+    (property "Sheetname" "")
+    (property "ki_description" "Generic connector, double row, 02x18, odd/even pin numbering scheme (row 1 odd numbers, row 2 even numbers), script generated (kicad-library-utils/schlib/autogen/connector/)")
+    (property "ki_keywords" "connector")
+    (attr through_hole)
+    (fp_text reference "P1" (at 0 -0.5 -90 unlocked) (layer "F.SilkS")
+        (effects (font (size 1 1) (thickness 0.1)))
+    )
+    (fp_text value "Cartridge Slot" (at 0 1 -90 unlocked) (layer "F.Fab")
+        (effects (font (size 1 1) (thickness 0.15)))
+    )
+    (fp_text user "Front of Cartridge" (at 14.732 4.826 -90 unlocked) (layer "F.SilkS")
+        (effects (font (size 1 1) (thickness 0.1)) (justify left bottom))
+    )
+    (fp_text user "${REFERENCE}" (at 0 2.5 -90 unlocked) (layer "F.Fab")
+        (effects (font (size 1 1) (thickness 0.15)))
+    )
+    (pad "1" thru_hole circle (at 0 0 270) (size 2 2) (drill 1.3) (layers "*.Cu" "*.Mask")
+      (net 3 "+5V") (pinfunction "Pin_1") (pintype "passive"))
+    (pad "2" thru_hole circle (at 0 -4.85 270) (size 2 2) (drill 1.3) (layers "*.Cu" "*.Mask")
+      (net 15 "-5V") (pinfunction "Pin_2") (pintype "passive"))
+    (pad "3" thru_hole circle (at 2.54 0 270) (size 2 2) (drill 1.3) (layers "*.Cu" "*.Mask")
+      (net 105 "/a8") (pinfunction "Pin_3") (pintype "passive"))
+    (pad "4" thru_hole circle (at 2.54 -4.85 270) (size 2 2) (drill 1.3) (layers "*.Cu" "*.Mask")
+      (net 106 "/a9") (pinfunction "Pin_4") (pintype "passive"))
+    (pad "5" thru_hole circle (at 5.08 0) (size 2 2) (drill 1.3) (layers "*.Cu" "*.Mask")
+      (net 103 "/a6") (pinfunction "Pin_5") (pintype "passive"))
+    (pad "6" thru_hole circle (at 5.08 -4.85 90) (size 2 2) (drill 1.3) (layers "*.Cu" "*.Mask")
+      (net 104 "/a7") (pinfunction "Pin_6") (pintype "passive"))
+    (pad "7" thru_hole circle (at 7.62 0) (size 2 2) (drill 1.3) (layers "*.Cu" "*.Mask")
+      (net 101 "/a4") (pinfunction "Pin_7") (pintype "passive"))
+    (pad "8" thru_hole circle (at 7.62 -4.85 90) (size 2 2) (drill 1.3) (layers "*.Cu" "*.Mask")
+      (net 102 "/a5") (pinfunction "Pin_8") (pintype "passive"))
+    (pad "9" thru_hole circle (at 10.16 0) (size 2 2) (drill 1.3) (layers "*.Cu" "*.Mask")
+      (net 99 "/a2") (pinfunction "Pin_9") (pintype "passive"))
+    (pad "10" thru_hole circle (at 10.16 -4.85 90) (size 2 2) (drill 1.3) (layers "*.Cu" "*.Mask")
+      (net 100 "/a3") (pinfunction "Pin_10") (pintype "passive"))
+    (pad "11" thru_hole circle (at 12.7 0) (size 2 2) (drill 1.3) (layers "*.Cu" "*.Mask")
+      (net 97 "/a0") (pinfunction "Pin_11") (pintype "passive"))
+    (pad "12" thru_hole circle (at 12.7 -4.85 90) (size 2 2) (drill 1.3) (layers "*.Cu" "*.Mask")
+      (net 98 "/a1") (pinfunction "Pin_12") (pintype "passive"))
+    (pad "13" thru_hole circle (at 15.24 0) (size 2 2) (drill 1.3) (layers "*.Cu" "*.Mask")
+      (net 51 "/a11") (pinfunction "Pin_13") (pintype "passive"))
+    (pad "14" thru_hole circle (at 15.24 -4.85 90) (size 2 2) (drill 1.3) (layers "*.Cu" "*.Mask")
+      (net 107 "/a10") (pinfunction "Pin_14") (pintype "passive"))
+    (pad "15" thru_hole circle (at 17.78 0 90) (size 2 2) (drill 1.3) (layers "*.Cu" "*.Mask")
+      (net 109 "/a13") (pinfunction "Pin_15") (pintype "passive"))
+    (pad "16" thru_hole circle (at 17.78 -4.85 90) (size 2 2) (drill 1.3) (layers "*.Cu" "*.Mask")
+      (net 108 "/a12") (pinfunction "Pin_16") (pintype "passive"))
+    (pad "17" thru_hole circle (at 20.32 0 90) (size 2 2) (drill 1.3) (layers "*.Cu" "*.Mask")
+      (net 111 "/a15") (pinfunction "Pin_17") (pintype "passive"))
+    (pad "18" thru_hole circle (at 20.32 -4.85 90) (size 2 2) (drill 1.3) (layers "*.Cu" "*.Mask")
+      (net 110 "/a14") (pinfunction "Pin_18") (pintype "passive"))
+    (pad "19" thru_hole circle (at 22.86 0 90) (size 2 2) (drill 1.3) (layers "*.Cu" "*.Mask")
+      (net 116 "/d3") (pinfunction "Pin_19") (pintype "passive"))
+    (pad "20" thru_hole circle (at 22.86 -4.85 90) (size 2 2) (drill 1.3) (layers "*.Cu" "*.Mask")
+      (net 117 "/d2") (pinfunction "Pin_20") (pintype "passive"))
+    (pad "21" thru_hole circle (at 25.4 0 90) (size 2 2) (drill 1.3) (layers "*.Cu" "*.Mask")
+      (net 118 "/d1") (pinfunction "Pin_21") (pintype "passive"))
+    (pad "22" thru_hole circle (at 25.4 -4.85 90) (size 2 2) (drill 1.3) (layers "*.Cu" "*.Mask")
+      (net 119 "/d0") (pinfunction "Pin_22") (pintype "passive"))
+    (pad "23" thru_hole circle (at 27.94 0 90) (size 2 2) (drill 1.3) (layers "*.Cu" "*.Mask")
+      (net 115 "/d4") (pinfunction "Pin_23") (pintype "passive"))
+    (pad "24" thru_hole circle (at 27.94 -4.85 90) (size 2 2) (drill 1.3) (layers "*.Cu" "*.Mask")
+      (net 114 "/d5") (pinfunction "Pin_24") (pintype "passive"))
+    (pad "25" thru_hole circle (at 30.48 0 90) (size 2 2) (drill 1.3) (layers "*.Cu" "*.Mask")
+      (net 113 "/d6") (pinfunction "Pin_25") (pintype "passive"))
+    (pad "26" thru_hole circle (at 30.48 -4.85 90) (size 2 2) (drill 1.3) (layers "*.Cu" "*.Mask")
+      (net 68 "/Φ2") (pinfunction "Pin_26") (pintype "passive"))
+    (pad "27" thru_hole circle (at 33.02 0 90) (size 2 2) (drill 1.3) (layers "*.Cu" "*.Mask")
+      (net 120 "/R{slash}~{W}") (pinfunction "Pin_27") (pintype "passive"))
+    (pad "28" thru_hole circle (at 33.02 -4.85 90) (size 2 2) (drill 1.3) (layers "*.Cu" "*.Mask")
+      (net 112 "/d7") (pinfunction "Pin_28") (pintype "passive"))
+    (pad "29" thru_hole circle (at 35.56 0 90) (size 2 2) (drill 1.3) (layers "*.Cu" "*.Mask")
+      (net 145 "/~{ROM1}") (pinfunction "Pin_29") (pintype "passive"))
+    (pad "30" thru_hole circle (at 35.56 -4.85 90) (size 2 2) (drill 1.3) (layers "*.Cu" "*.Mask")
+      (net 4 "/AUDIO_IN") (pinfunction "Pin_30") (pintype "passive"))
+    (pad "31" thru_hole circle (at 38.1 0 90) (size 2 2) (drill 1.3) (layers "*.Cu" "*.Mask")
+      (net 57 "/~{WRAM_CE}") (pinfunction "Pin_31") (pintype "passive"))
+    (pad "32" thru_hole circle (at 38.1 -4.85 90) (size 2 2) (drill 1.3) (layers "*.Cu" "*.Mask")
+      (net 146 "/~{ROM2}") (pinfunction "Pin_32") (pintype "passive"))
+    (pad "33" thru_hole circle (at 40.64 0 90) (size 2 2) (drill 1.3) (layers "*.Cu" "*.Mask")
+      (net 144 "/~{ROM0}") (pinfunction "Pin_33") (pintype "passive"))
+    (pad "34" thru_hole circle (at 40.64 -4.85 90) (size 2 2) (drill 1.3) (layers "*.Cu" "*.Mask")
+      (net 148 "/~{ROM_RD}") (pinfunction "Pin_34") (pintype "passive"))
+    (pad "35" thru_hole circle (at 43.18 0 90) (size 2 2) (drill 1.3) (layers "*.Cu" "*.Mask")
+      (net 2 "GND") (pinfunction "Pin_35") (pintype "passive"))
+    (pad "36" thru_hole circle (at 43.18 -4.85 90) (size 2 2) (drill 1.3) (layers "*.Cu" "*.Mask")
+      (net 13 "+12V") (pinfunction "Pin_36") (pintype "passive"))
   )
   (footprint "Diode_THT:D_DO-35_SOD27_P7.62mm_Horizontal" (layer "F.Cu")
@@
   (segment (start 184.811929 54.865) (end 186.183 53.493929) (width 0.25) (layer "F.Cu") (net 64))
   (segment (start 78.4 58.457929) (end 78.4 59.032929) (width 0.75) (layer "B.Cu") (net 65))
-  (segment (start 77.725 133.503929) (end 77.725 59.707929) (width 0.75) (layer "B.Cu") (net 65))
   (segment (start 77.725 139.472929) (end 77.725 133.503929) (width 0.75) (layer "B.Cu") (net 65))
   (segment (start 78.4 59.032929) (end 77.725 59.707929) (width 0.75) (layer "B.Cu") (net 65))
