File: creativision-clone.kicad_pcb (KiCad board)
At the start: 2 copper layers, 208.8 x 99.7 mm, 105 parts, among them J1 Conn_01x10_Socket, J2 Conn_01x10_Socket, J3 Conn_01x07_Pin, J4 Conn_01x04_Socket, J5 RCJ-013, J6 RCJ-014, P1 Cartridge Slot, Q1 2n4401, SW1 Reset, SW2 Power Toggle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

Commit message: Move caps for guaranteed x-clearance
Parts:
- moved C12 7.91 mm to (101.4, 124.9)
- moved C13 7.91 mm to (93.2, 124.9)
- moved TP1 5.80 mm to (103.1, 131.2)
Routing:
- net +5V: track 556.1 -> 533.0 mm
- net /SW_VCC: track 14.6 -> 22.5 mm, vias 0 -> 1
- net /a7: track 204.4 -> 206.5 mm
Changed lines of the file:
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@@
   )
   (footprint "TestPoint:TestPoint_Loop_D2.50mm_Drill1.0mm" (layer "F.Cu")
-    (at 98.045 128.423929)
+    (at 103.125 131.217929)
     (descr "wire loop as test point, loop diameter 2.5mm, hole diameter 1.0mm")
     (tags "test point wire loop bead")
@@
   )
   (footprint "Capacitor_THT:CP_Radial_D6.3mm_P2.50mm" (layer "F.Cu")
-    (at 85.305 124.867929 180)
+    (at 93.219 124.867929 180)
     (descr "CP, Radial series, Radial, pin pitch=2.50mm, , diameter=6.3mm, Electrolytic Capacitor")
     (tags "CP Radial series Radial pin pitch 2.50mm  diameter 6.3mm Electrolytic Capacitor")
@@
   )
   (footprint "Capacitor_THT:CP_Radial_D6.3mm_P2.50mm" (layer "F.Cu")
-    (at 93.51238 124.867929 180)
+    (at 101.42638 124.867929 180)
     (descr "CP, Radial series, Radial, pin pitch=2.50mm, , diameter=6.3mm, Electrolytic Capacitor")
     (tags "CP Radial series Radial pin pitch 2.50mm  diameter 6.3mm Electrolytic Capacitor")
@@
   (segment (start 172.467 61.233) (end 174.645 59.055) (width 0.75) (layer "B.Cu") (net 2))
   (segment (start 177.165 113.03) (end 177.165 118.11) (width 0.75) (layer "B.Cu") (net 2))
-  (segment (start 93.51238 124.867929) (end 92.13738 126.242929) (width 0.75) (layer "F.Cu") (net 3))
   (segment (start 239.777 78.639929) (end 243.739929 78.639929) (width 0.75) (layer "F.Cu") (net 3))
   (segment (start 101.855 124.867929) (end 105.03 121.692929) (width 0.75) (layer "F.Cu") (net 3))
@@
   (segment (start 253.493 130.963929) (end 269.241 130.963929) (width 0.75) (layer "F.Cu") (net 3))
   (segment (start 253.593071 78.74) (end 253.747 78.893929) (width 0.75) (layer "F.Cu") (net 3))
-  (segment (start 86.68 126.242929) (end 85.305 124.867929) (width 0.75) (layer "F.Cu") (net 3))
   (segment (start 271.527 65.107) (end 270.428 64.008) (width 0.75) (layer "F.Cu") (net 3))
   (segment (start 253.238 122.936) (end 263.138071 122.936) (width 0.75) (layer "F.Cu") (net 3))
   (segment (start 118.745 72.39) (end 120.804929 72.39) (width 0.75) (layer "F.Cu") (net 3))
-  (segment (start 92.13738 126.242929) (end 86.68 126.242929) (width 0.75) (layer "F.Cu") (net 3))
   (segment (start 156.21 59.69) (end 152.908 59.69) (width 0.75) (layer "F.Cu") (net 3))
   (segment (start 208.43 116.634929) (end 199.286 116.634929) (width 0.75) (layer "F.Cu") (net 3))
@@
   (segment (start 163.831 72.289929) (end 165.609 72.289929) (width 0.75) (layer "F.Cu") (net 3))
   (segment (start 254.255 62.383929) (end 266.853929 62.383929) (width 0.75) (layer "F.Cu") (net 3))
-  (segment (start 98.045 128.677929) (end 101.855 124.867929) (width 0.75) (layer "F.Cu") (net 3))
   (segment (start 119.099071 66.955929) (end 118.745 67.31) (width 0.75) (layer "F.Cu") (net 3))
   (segment (start 271.527 128.677929) (end 271.527 65.107) (width 0.75) (layer "F.Cu") (net 3))
@@
   (segment (start 199.286 116.634929) (end 199.137 116.485929) (width 0.75) (layer "F.Cu") (net 3))
   (segment (start 253.239 130.709929) (end 253.493 130.963929) (width 0.75) (layer "F.Cu") (net 3))
-  (segment (start 93.51238 124.867929) (end 101.855 124.867929) (width 0.75) (layer "F.Cu") (net 3))
   (segment (start 243.739929 78.639929) (end 243.84 78.74) (width 0.75) (layer "F.Cu") (net 3))
   (segment (start 105.03 126.140721) (end 105.03 121.692929) (width 0.75) (layer "F.Cu") (net 3))
@@
   (via (at 161.291 129.439929) (size 0.8) (drill 0.4) (layers "F.Cu" "B.Cu") (net 104))
   (via (at 94.235 76.861929) (size 0.8) (drill 0.4) (layers "F.Cu" "B.Cu") (net 104))
-  (segment (start 98.045 120.295929) (end 106.427 128.677929) (width 0.25) (layer "B.Cu") (net 104))
   (segment (start 94.235 76.861929) (end 94.235 119.787929) (width 0.25) (layer "B.Cu") (net 104))
+  (segment (start 100.05138 125.742929) (end 100.05138 122.302309) (width 0.25) (layer "B.Cu") (net 104))
+  (segment (start 102.98638 128.677929) (end 100.05138 125.742929) (width 0.25) (layer "B.Cu") (net 104))
+  (segment (start 100.05138 122.302309) (end 98.045 120.295929) (width 0.25) (layer "B.Cu") (net 104))
   (segment (start 94.235 119.787929) (end 94.489 120.041929) (width 0.25) (layer "B.Cu") (net 104))
   (segment (start 160.8 128.948929) (end 160.8 103.995) (width 0.25) (layer "B.Cu") (net 104))
   (segment (start 160.8 103.995) (end 161.925 102.87) (width 0.25) (layer "B.Cu") (net 104))
+  (segment (start 108.967 128.677929) (end 102.98638 128.677929) (width 0.25) (layer "B.Cu") (net 104))
   (segment (start 161.291 129.439929) (end 160.8 128.948929) (width 0.25) (layer "B.Cu") (net 104))
-  (segment (start 106.427 128.677929) (end 108.967 128.677929) (width 0.25) (layer "B.Cu") (net 104))
   (segment (start 163.34 106.825) (end 179.004402 106.825) (width 0.25) (layer "F.Cu") (net 105))
   (segment (start 182.245 100.33) (end 186.055 100.33) (width 0.25) (layer "F.Cu") (net 105))
@@
   (segment (start 266.7 97.155) (end 266.7 128.27) (width 0.25) (layer "B.Cu") (net 153))
   (segment (start 266.065 74.295) (end 266.065 96.52) (width 0.25) (layer "B.Cu") (net 153))
+  (segment (start 90.719 124.867929) (end 82.805 124.867929) (width 0.75) (layer "F.Cu") (net 158))
+  (via (at 82.805 124.867929) (size 0.8) (drill 0.4) (layers "F.Cu" "B.Cu") (net 158))
   (segment (start 82.805 139.472929) (end 82.805 124.867929) (width 0.75) (layer "B.Cu") (net 158))
   (zone (net 3) (net_name "+5V") (layer "F.Cu") (hatch edge 0.5)
