File: v1-creativision-snes-pcb/v1-creativision-snes-pcb.kicad_sch (KiCad schematic)
At the start: 14 parts, among them J1 Left Joystick, J2 Right Joystick, J4 PS/2 Keyboard, J5 SNES, J6 Debug, SW1 Reset Pico, U1 Pico, U2 LOGIC-SN74LVC245AN(DIP20-7.62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, U3 LOGIC-SN74LVC245AN(DIP20-7.62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

Commit message: Add diode to prevent backpowering when uploading firmware
Parts:
- added D1: D, Diode_THT:D_DO-15_P10.16mm_Horizontal, symbol Device:D
Connections:
- net +5V: now also D1.2 (A); no longer U1.39 (VSYS)
- new net: D1.1 (K), U1.39 (VSYS)

Commit message: Fix DIR pin error
Parts:
- removed J6: Debug, Connector_PinHeader_2.54mm:PinHeader_1x03_P2.54mm_Vertical, symbol Connector:Conn_01x03_Pin
- added C1: 220µF, Capacitor_THT:CP_Radial_D6.3mm_P2.50mm, symbol Device:C_Polarized_Small
Connections:
- net +3.3V: no longer JP1.2 (B), JP2.2 (B)
- net +5V: now also C1.1
- net GND: now also JP1.2 (B), JP2.2 (B), C1.2; no longer U1.42 (GND)
- net SWCLK: no longer names the net of U1.41 (SWCLK)
- net SWDIO: no longer names the net of U1.43 (SWDIO)
- no-connect marks 6 -> 9
Other:
- moved on the sheet: JP1, JP2
